Commit message: house cleaning

File: urdf/expanded_xacro.urdf (robot description, URDF)
Before this commit: robot enesbot_dualarm_v0.1, 15 links, 14 joints
Links:
- link l1: geometry visual mesh filename=package://enesbot_dualarm/meshes/n1.stl
- link l2: geometry visual mesh filename=package://enesbot_dualarm/meshes/n0.stl
- link l3: geometry visual mesh filename=package://enesbot_dualarm/meshes/n1.stl
- link l4: geometry visual mesh filename=package://enesbot_dualarm/meshes/n0.stl
- link l5: geometry visual mesh filename=package://enesbot_dualarm/meshes/n1.stl
- link l6: geometry visual mesh filename=package://enesbot_dualarm/meshes/n0.stl
- link l7: geometry visual mesh filename=package://enesbot_dualarm/meshes/n2.stl
- link map: geometry visual mesh filename=package://enesbot_dualarm/meshes/nb.stl
- link r1: geometry visual mesh filename=package://enesbot_dualarm/meshes/n1.stl
- link r2: geometry visual mesh filename=package://enesbot_dualarm/meshes/n0.stl
- link r3: geometry visual mesh filename=package://enesbot_dualarm/meshes/n1.stl
- link r4: geometry visual mesh filename=package://enesbot_dualarm/meshes/n0.stl
- link r5: geometry visual mesh filename=package://enesbot_dualarm/meshes/n1.stl
- link r6: geometry visual mesh filename=package://enesbot_dualarm/meshes/n0.stl
- link r7: geometry visual mesh filename=package://enesbot_dualarm/meshes/n2.stl
