Commit message: changed 'map' link to 'root'

File: urdf/enesbot_dualarm.xacro (robot description, xacro)
@@ -21,5 +21,5 @@
     </link>
   </xacro:macro>
-	<link name="map">
+	<link name="root">
 		<visual>
 			<geometry>
@@ -28,5 +28,5 @@
 		</visual>
 	</link>
-  <xacro:segment n="r1" parent="map" child="r1"   cad_type="1" xyz="1 0 0" origin="0 -0.15 0.4" rpy="0 -0.523599 -0.523599" />
+  <xacro:segment n="r1" parent="root" child="r1"   cad_type="1" xyz="1 0 0" origin="0 -0.15 0.4" rpy="0 -0.523599 -0.523599" />
   <xacro:segment n="r2" parent="r1"  child="r2"   cad_type="0" xyz="0 0 1" origin="0.1 0 0" rpy="0 0 0" />
   <xacro:segment n="r3" parent="r2"  child="r3"   cad_type="1" xyz="1 0 0" origin="0.1 0 0" rpy="0 0 0" />
@@ -35,5 +35,5 @@
   <xacro:segment n="r6" parent="r5"  child="r6"   cad_type="0" xyz="0 0 1" origin="0.1 0 0" rpy="0 0 0" />
   <xacro:segment n="r7" parent="r6"  child="r7"   cad_type="2" xyz="1 0 0" origin="0.1 0 0" rpy="0 0 0" />
-  <xacro:segment n="l1" parent="map" child="l1"   cad_type="1" xyz="1 0 0" origin="0 0.15 0.4" rpy="0 -0.523599 0.523599" />
+  <xacro:segment n="l1" parent="root" child="l1"   cad_type="1" xyz="1 0 0" origin="0 0.15 0.4" rpy="0 -0.523599 0.523599" />
   <xacro:segment n="l2" parent="l1"  child="l2"   cad_type="0" xyz="0 0 1" origin="0.1 0 0" rpy="0 0 0" />
   <xacro:segment n="l3" parent="l2"  child="l3"   cad_type="1" xyz="1 0 0" origin="0.1 0 0" rpy="0 0 0" />

File: urdf/exp_enesbot_dualarm.urdf (robot description, URDF)
Before this commit: robot enesbot_dualarm, 15 links, 14 joints
Links:
- removed link map
- added link root; visual mesh filename=package://enesbot_dualarm/meshes/nb.stl
Joints:
- joint jl1: parent map -> root
- joint jr1: parent map -> root
